File: board/operator-mk2/operator-mk2.kicad_pcb (KiCad board)
At the start: 2 copper layers, 64 x 28 mm, 11 parts, among them J1 Slide Switch, J2 Microphone, J3 Buttons, J4 Speaker, J5 Xiao Left, J6 Xiao Right, J8 TRRS Socket

Commit message: archive
Routing:
- net BCLK: track 57.5 -> 54.1 mm
Changed lines of the file:
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@@
 	)
 	(segment
-		(start 155.649 105.901024)
-		(end 155.649 104.211)
+		(start 134 99)
+		(end 142.5 107.5)
 		(width 0.4)
 		(layer "F.Cu")
@@
 	)
 	(segment
-		(start 155.649 104.211)
-		(end 157.1 102.76)
+		(start 148.76 107.5)
+		(end 153.5 102.76)
+		(width 0.4)
+		(layer "F.Cu")
+		(net 2)
+	)
+	(segment
+		(start 134 92.56)
+		(end 134 99)
+		(width 0.4)
+		(layer "F.Cu")
+		(net 2)
+	)
+	(segment
+		(start 142.5 107.5)
+		(end 148.76 107.5)
 		(width 0.4)
 		(layer "F.Cu")
@@
 		(width 0.4)
 		(layer "F.Cu")
-		(net 2)
-	)
-	(segment
-		(start 142.633976 106.751)
-		(end 154.799024 106.751)
-		(width 0.4)
-		(layer "F.Cu")
-		(net 2)
-	)
-	(segment
-		(start 134 92.56)
-		(end 134 98.117024)
-		(width 0.4)
-		(layer "F.Cu")
-		(net 2)
-	)
-	(segment
-		(start 134 98.117024)
-		(end 142.633976 106.751)
-		(width 0.4)
-		(layer "F.Cu")
-		(net 2)
-	)
-	(segment
-		(start 154.799024 106.751)
-		(end 155.649 105.901024)
-		(width 0.4)
-		(layer "F.Cu")
