File: board/audio-breakout-mk2/audio-breakout-mk2.kicad_pcb (KiCad board)
At the start: 2 copper layers, 24 x 21 mm, 2 parts, among them J1 Conn_01x06_Socket

Commit message: audio board mk2
Parts:
- added REF**: MountingHole_3.2mm_M3, MountingHole:MountingHole_3.2mm_M3, F.Cu at (130.0, 70.0)
- added REF**: MountingHole_3.2mm_M3, MountingHole:MountingHole_3.2mm_M3, F.Cu at (154.0, 70.0)
- Socket1: renamed from J1; footprint Connector_PinSocket_2.54mm:PinSocket_1x06_P2.54mm_Vertical -> Connector_PinHeader_2.54mm:PinHeader_1x06_P2.54mm_Vertical_SMD_Pin1Left
- moved Socket1 6.46 mm to (142.0, 83.1)
- renumbered MK1 to MK2
Connections:
- MK2 pad 1: Net-(J1-Pin_1) -> Net-(MK1-WS)
- MK2 pad 2: Net-(J1-Pin_2) -> Net-(MK1-LR)
- MK2 pad 5: Net-(J1-Pin_5) -> Net-(MK1-VDD)
- MK2 pad 6: Net-(J1-Pin_6) -> Net-(MK1-SD)
- Socket1 pad 1: Net-(J1-Pin_1) -> Net-(MK1-LR)
- Socket1 pad 2: Net-(J1-Pin_2) -> Net-(MK1-WS)
- Socket1 pad 3: GND -> Net-(MK1-SD)
- Socket1 pad 5: Net-(J1-Pin_5) -> GND
- Socket1 pad 6: Net-(J1-Pin_6) -> Net-(MK1-VDD)
Routing:
- net Net-(MK1-SD): track 0.00 -> 39.9 mm
- net Net-(MK1-WS): track 0.00 -> 33.3 mm
- net Net-(J1-Pin_6): track 19.9 -> 0.00 mm
- net Net-(J1-Pin_1): track 14.9 -> 0.00 mm
- net Net-(J1-Pin_5): track 14.0 -> 0.00 mm
- net Net-(MK1-LR): track 0.00 -> 13.5 mm
- net Net-(MK1-VDD): track 0.00 -> 12.9 mm
- net Net-(J1-Pin_2): track 12.6 -> 0.00 mm
- net Net-(MK1-SCK): track 12.1 -> 9.63 mm
Other:
- board size 24 x 21 mm -> 32 x 24 mm

Commit message: save
Parts:
- removed the REF** at (130.0, 70.0)
- removed the REF** at (154.0, 70.0)
- added REF**: MountingHole_M3, Fab:MountingHole_M3, F.Cu at (130.0, 70.0)
- added REF**: MountingHole_M3, Fab:MountingHole_M3, F.Cu at (154.0, 70.0)
Changed lines of the file:
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@@
 	(net 5 "Net-(MK1-SCK)")
 	(net 6 "Net-(MK1-VDD)")
-	(footprint "MountingHole:MountingHole_3.2mm_M3"
-		(layer "F.Cu")
-		(at 130 70)
-		(descr "Mounting Hole 3.2mm, no annular, M3")
-		(tags "mounting hole 3.2mm no annular m3")
-		(property "Reference" "REF**"
-			(at 0 -4.2 0)
-			(layer "F.SilkS")
-			(hide yes)
-			(effects
-				(font
-					(size 1 1)
-					(thickness 0.15)
-				)
-			)
-		)
-		(property "Value" "MountingHole_3.2mm_M3"
-			(at 6 -6 0)
-			(layer "F.Fab")
-			(hide yes)
-			(effects
-				(font
-					(size 1 1)
-					(thickness 0.15)
-				)
-			)
-		)
-		(property "Datasheet" ""
-			(at 0 0 0)
-			(layer "F.Fab")
-			(hide yes)
-			(effects
-				(font
-					(size 1.27 1.27)
-					(thickness 0.15)
-				)
-			)
-		)
-		(property "Description" ""
-			(at 0 0 0)
-			(layer "F.Fab")
-			(hide yes)
-			(effects
-				(font
-					(size 1.27 1.27)
-					(thickness 0.15)
-				)
-			)
-		)
-		(attr exclude_from_pos_files exclude_from_bom)
-		(fp_circle
-			(center 0 0)
-			(end 3.2 0)
-			(stroke
-				(width 0.15)
-				(type solid)
-			)
-			(fill no)
-			(layer "Cmts.User")
-		)
-		(fp_circle
-			(center 0 0)
-			(end 3.45 0)
-			(stroke
-				(width 0.05)
-				(type solid)
-			)
-			(fill no)
-			(layer "F.CrtYd")
-		)
-		(pad "" np_thru_hole circle
-			(at 0 0)
-			(size 3.2 3.2)
-			(drill 3.2)
-			(layers "*.Cu" "*.Mask")
-		)
-		(embedded_fonts no)
-	)
 	(footprint "Connector_PinHeader_2.54mm:PinHeader_1x06_P2.54mm_Vertical_SMD_Pin1Left"
 		(layer "F.Cu")
@@
 			)
 		)
+	)
+	(footprint "Fab:MountingHole_M3"
+		(layer "F.Cu")
+		(at 130 70)
+		(property "Reference" "REF**"
+			(at 0 3 0)
+			(layer "F.SilkS")
+			(hide yes)
+			(effects
+				(font
+					(size 1 1)
+					(thickness 0.15)
+				)
+			)
+		)
+		(property "Value" "MountingHole_M3"
+			(at 0 -3 0)
+			(layer "F.Fab")
+			(hide yes)
+			(effects
+				(font
+					(size 1 1)
+					(thickness 0.15)
+				)
+			)
+		)
+		(property "Datasheet" ""
+			(at 0 0 0)
+			(layer "F.Fab")
+			(hide yes)
+			(effects
+				(font
+					(size 1.27 1.27)
+					(thickness 0.15)
+				)
+			)
+		)
+		(property "Description" ""
+			(at 0 0 0)
+			(layer "F.Fab")
+			(hide yes)
+			(effects
+				(font
+					(size 1.27 1.27)
+					(thickness 0.15)
+				)
+			)
+		)
+		(attr through_hole)
+		(fp_text user "M3"
+			(at 0 0 0)
+			(unlocked yes)
+			(layer "F.Fab")
+			(effects
+				(font
+					(size 0.5 0.5)
+					(thickness 0.1)
+				)
+			)
+		)
+		(pad "" thru_hole circle
+			(at 0 0)
+			(size 3.3 3.3)
+			(drill 3.1)
+			(layers "*.Cu" "*.Mask")
+			(remove_unused_layers no)
+		)
+		(embedded_fonts no)
 	)
 	(footprint "fab:Mic_MEMS_TDK_ICS-43434"
@@
 		)
 	)
-	(footprint "MountingHole:MountingHole_3.2mm_M3"
+	(footprint "Fab:MountingHole_M3"
 		(layer "F.Cu")
 		(at 154 70)
-		(descr "Mounting Hole 3.2mm, no annular, M3")
-		(tags "mounting hole 3.2mm no annular m3")
 		(property "Reference" "REF**"
-			(at 0 -4.2 0)
+			(at 0 3 0)
 			(layer "F.SilkS")
 			(hide yes)
@@
 			)
 		)
-		(property "Value" "MountingHole_3.2mm_M3"
-			(at -6 -5 0)
+		(property "Value" "MountingHole_M3"
+			(at 0 -3 0)
 			(layer "F.Fab")
 			(hide yes)
@@
 			)
 		)
-		(attr exclude_from_pos_files exclude_from_bom)
-		(fp_circle
-			(center 0 0)
-			(end 3.2 0)
-			(stroke
-				(width 0.15)
-				(type solid)
-			)
-			(fill no)
-			(layer "Cmts.User")
-		)
-		(fp_circle
-			(center 0 0)
-			(end 3.45 0)
-			(stroke
-				(width 0.05)
-				(type solid)
-			)
-			(fill no)
-			(layer "F.CrtYd")
-		)
-		(pad "" np_thru_hole circle
+		(attr through_hole)
+		(fp_text user "M3"
+			(at 0 0 0)
+			(unlocked yes)
+			(layer "F.Fab")
+			(effects
+				(font
+					(size 0.5 0.5)
+					(thickness 0.1)
+				)
+			)
+		)
+		(pad "" thru_hole circle
 			(at 0 0)
-			(size 3.2 3.2)
-			(drill 3.2)
+			(size 3.3 3.3)
+			(drill 3.1)
 			(layers "*.Cu" "*.Mask")
+			(remove_unused_layers no)
 		)
 		(embedded_fonts no)
