File: board/operator-mk3/_autosave-operator-mk3.kicad_pcb (KiCad board)
At the start: 2 copper layers, 57 x 28 mm, 11 parts, among them J1 Slide Switch, J2 Microphone, J3 Buttons, J4 Speaker, J5 Xiao Left, J6 Xiao Right, J8 TRRS Socket

Commit message: update notes
Routing:
- added copper zone on F.Cu, net GND
- removed copper zone on F.Cu, net (none)
Changed lines of the file:
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@@
+	)
+	(segment
+		(start 141 109)
+		(end 131.5 99.5)
+		(width 0.6)
+		(layer "F.Cu")
+		(net 4)
 	)
 	(segment
 		(start 156.7 109)
 		(end 141 109)
-		(width 0.6)
-		(layer "F.Cu")
-		(net 4)
-	)
-	(segment
-		(start 141 109)
-		(end 131.5 99.5)
 		(width 0.6)
 		(layer "F.Cu")
@@
 	)
 	(segment
+		(start 123.5 95)
+		(end 118.28 100.22)
+		(width 0.6)
+		(layer "B.Cu")
+		(net 4)
+	)
+	(segment
 		(start 153.5 105.8)
 		(end 153.5 105.3)
 		(width 0.8)
-		(layer "B.Cu")
-		(net 4)
-	)
-	(segment
-		(start 123.5 95)
-		(end 118.28 100.22)
-		(width 0.6)
 		(layer "B.Cu")
 		(net 4)
@@
 	)
 	(zone
-		(net 0)
-		(net_name "")
+		(net 3)
+		(net_name "GND")
 		(layer "F.Cu")
 		(hatch edge 0.5)
@@
 			(thermal_gap 0.5)
 			(thermal_bridge_width 0.5)
-			(island_removal_mode 1)
-			(island_area_min 10)
 		)
 		(polygon
