File: board/switchboard-mk4/switchboard-mk4.kicad_pcb (KiCad board)
At the start: 2 copper layers, 63 x 37 mm, 21 parts, among them J1 Socket 02, J10 Xiao Left, J2 Socket 03, J3 Socket 01, J4 Socket 06, J5 Socket 05, J6 Socket 04, J7 Socket 07, J8 Socket 08, J9 Xiao Right

Commit message: add new board design
Parts:
- removed the REF** at (199.5, 61.0)
- removed the REF** at (171.0, 92.0)
- removed the REF** at (228.0, 92.0)
- added REF**: MountingHole_M3, fab:MountingHole_M3, F.Cu at (228.0, 92.0)
- added REF**: MountingHole_M3, fab:MountingHole_M3, F.Cu at (199.5, 61.0)
- added REF**: MountingHole_M3, fab:MountingHole_M3, F.Cu at (171.0, 92.0)
Changed lines of the file:
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@@
 		)
 	)
-	(footprint "fab:MountingHole_M2"
+	(footprint "fab:MountingHole_M3"
 		(layer "F.Cu")
-		(at 199.5 61)
+		(at 228 92)
 		(property "Reference" "REF**"
-			(at 0 2 0)
-			(layer "F.SilkS")
-			(hide yes)
-			(effects
-				(font
-					(size 1 1)
-					(thickness 0.15)
-				)
-			)
-		)
-		(property "Value" "MountingHole_M2"
-			(at 0 -2 0)
+			(at 0 3 0)
+			(layer "F.SilkS")
+			(hide yes)
+			(effects
+				(font
+					(size 1 1)
+					(thickness 0.15)
+				)
+			)
+		)
+		(property "Value" "MountingHole_M3"
+			(at 0 -3 0)
 			(layer "F.Fab")
 			(hide yes)
@@
 		)
 		(attr through_hole)
-		(fp_text user "M2"
+		(fp_text user "M3"
+			(at 2 0 0)
+			(unlocked yes)
+			(layer "F.SilkS")
+			(effects
+				(font
+					(size 1 1)
+					(thickness 0.15)
+					(bold yes)
+				)
+				(justify left)
+			)
+		)
+		(fp_text user "M3"
 			(at 0 0 0)
 			(unlocked yes)
@@
 		(pad "" thru_hole circle
 			(at 0 0)
-			(size 2.3 2.3)
-			(drill 2.1)
+			(size 3.3 3.3)
+			(drill 3.1)
 			(layers "*.Cu" "*.Mask")
 			(remove_unused_layers no)
@@
 		)
 	)
-	(footprint "fab:MountingHole_M2"
+	(footprint "fab:MountingHole_M3"
 		(layer "F.Cu")
-		(at 171 92)
+		(at 199.5 61)
 		(property "Reference" "REF**"
-			(at 0 2 0)
-			(layer "F.SilkS")
-			(hide yes)
-			(effects
-				(font
-					(size 1 1)
-					(thickness 0.15)
-				)
-			)
-		)
-		(property "Value" "MountingHole_M2"
-			(at 0 -2 0)
+			(at 0 3 0)
+			(layer "F.SilkS")
+			(hide yes)
+			(effects
+				(font
+					(size 1 1)
+					(thickness 0.15)
+				)
+			)
+		)
+		(property "Value" "MountingHole_M3"
+			(at 0 -3 0)
 			(layer "F.Fab")
 			(hide yes)
@@
 		)
 		(attr through_hole)
-		(fp_text user "M2"
+		(fp_text user "M3"
+			(at 2 0 0)
+			(unlocked yes)
+			(layer "F.SilkS")
+			(effects
+				(font
+					(size 1 1)
+					(thickness 0.15)
+					(bold yes)
+				)
+				(justify left)
+			)
+		)
+		(fp_text user "M3"
 			(at 0 0 0)
 			(unlocked yes)
@@
 		(pad "" thru_hole circle
 			(at 0 0)
-			(size 2.3 2.3)
-			(drill 2.1)
+			(size 3.3 3.3)
+			(drill 3.1)
 			(layers "*.Cu" "*.Mask")
 			(remove_unused_layers no)
@@
 		)
 	)
-	(footprint "fab:MountingHole_M2"
+	(footprint "fab:MountingHole_M3"
 		(layer "F.Cu")
-		(at 228 92)
+		(at 171 92)
 		(property "Reference" "REF**"
-			(at 0 2 0)
-			(layer "F.SilkS")
-			(hide yes)
-			(effects
-				(font
-					(size 1 1)
-					(thickness 0.15)
-				)
-			)
-		)
-		(property "Value" "MountingHole_M2"
-			(at 0 -2 0)
+			(at 0 3 0)
+			(layer "F.SilkS")
+			(hide yes)
+			(effects
+				(font
+					(size 1 1)
+					(thickness 0.15)
+				)
+			)
+		)
+		(property "Value" "MountingHole_M3"
+			(at 0 -3 0)
 			(layer "F.Fab")
 			(hide yes)
@@
 		)
 		(attr through_hole)
-		(fp_text user "M2"
+		(fp_text user "M3"
+			(at 2 0 0)
+			(unlocked yes)
+			(layer "F.SilkS")
+			(effects
+				(font
+					(size 1 1)
+					(thickness 0.15)
+					(bold yes)
+				)
+				(justify left)
+			)
+		)
+		(fp_text user "M3"
 			(at 0 0 0)
 			(unlocked yes)
@@
 		(pad "" thru_hole circle
 			(at 0 0)
-			(size 2.3 2.3)
-			(drill 2.1)
-			(layers "*.Cu" "*.Mask")
-			(remove_unused_layers no)
+			(size 3.3 3.3)
+			(drill 3.1)
+			(layers "*.Cu" "*.Mask")
+			(remove_unused_layers no)
